File: Temperature-Station_PCF8563/Mainboard1.1/Mainboard_1.1.sch (KiCad schematic (older format))
At the start: 34 parts, among them J1 CONN_01X03, J2 CONN_01X15, J3 CONN_01X15, J4 SD_Card, J5 CONN_01X03, J6 CONN_01X02, J7 CONN_01X02, J8 CONN_01X02, J9 CONN_01X02, U1 LM1117-3.3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

Commit message: Fixes
Added static/dhcp option for obtaining IP address
Little changes to code
Parts:
- added RJ8: 0, Resistors_SMD:R_1206_HandSoldering, symbol R
Connections:
- net GND: now also RJ8.1, RJ8.2
Changed lines of the file:
@@
 3V3
 $Comp
-L GND #PWR01
+L GND #PWR1
 U 1 1 591DCE28
 P 2600 1750
-F 0 "#PWR01" H 2600 1500 50  0001 C CNN
+F 0 "#PWR1" H 2600 1500 50  0001 C CNN
 F 1 "GND" H 2600 1600 50  0000 C CNN
 F 2 "" H 2600 1750 50  0001 C CNN
@@
 SCK
 $Comp
-L GND #PWR02
+L GND #PWR2
 U 1 1 591DCE55
 P 2600 2450
-F 0 "#PWR02" H 2600 2200 50  0001 C CNN
+F 0 "#PWR2" H 2600 2200 50  0001 C CNN
 F 1 "GND" H 2600 2300 50  0000 C CNN
 F 2 "" H 2600 2450 50  0001 C CNN
@@
 $EndComp
 $Comp
-L GND #PWR03
+L GND #PWR4
 U 1 1 591DD033
 P 3650 1750
-F 0 "#PWR03" H 3650 1500 50  0001 C CNN
+F 0 "#PWR4" H 3650 1500 50  0001 C CNN
 F 1 "GND" H 3650 1600 50  0000 C CNN
 F 2 "" H 3650 1750 50  0001 C CNN
@@
 3V3
 $Comp
-L GND #PWR04
+L GND #PWR5
 U 1 1 591DD05E
 P 3650 2150
-F 0 "#PWR04" H 3650 1900 50  0001 C CNN
+F 0 "#PWR5" H 3650 1900 50  0001 C CNN
 F 1 "GND" H 3650 2000 50  0000 C CNN
 F 2 "" H 3650 2150 50  0001 C CNN
@@
 1wire
 $Comp
-L GND #PWR05
+L GND #PWR15
 U 1 1 591DD301
 P 5200 2850
-F 0 "#PWR05" H 5200 2600 50  0001 C CNN
+F 0 "#PWR15" H 5200 2600 50  0001 C CNN
 F 1 "GND" H 5200 2700 50  0000 C CNN
 F 2 "" H 5200 2850 50  0001 C CNN
@@
 MOSI
 $Comp
-L GND #PWR06
+L GND #PWR16
 U 1 1 591DDAB3
 P 6500 2250
-F 0 "#PWR06" H 6500 2000 50  0001 C CNN
+F 0 "#PWR16" H 6500 2000 50  0001 C CNN
 F 1 "GND" H 6500 2100 50  0000 C CNN
 F 2 "" H 6500 2250 50  0001 C CNN
@@
 	0    1    1    0
 $EndComp
-Text GLabel 6500 2350 0    60   Input ~ 0
-3V3
 Text GLabel 6500 2450 0    60   Input ~ 0
 SCK
 $Comp
-L GND #PWR07
+L GND #PWR17
 U 1 1 591DDB59
 P 6500 2550
-F 0 "#PWR07" H 6500 2300 50  0001 C CNN
+F 0 "#PWR17" H 6500 2300 50  0001 C CNN
 F 1 "GND" H 6500 2400 50  0000 C CNN
 F 2 "" H 6500 2550 50  0001 C CNN
@@
 	1    0    0    -1
 $EndComp
-Text GLabel 9000 1850 1    60   Input ~ 0
-3V3
 Text GLabel 9050 2150 2    60   Input ~ 0
 SD_D
@@
 3V3
 $Comp
-L GND #PWR08
+L GND #PWR3
 U 1 1 591DF8F9
 P 3300 5600
-F 0 "#PWR08" H 3300 5350 50  0001 C CNN
+F 0 "#PWR3" H 3300 5350 50  0001 C CNN
 F 1 "GND" H 3300 5450 50  0000 C CNN
 F 2 "" H 3300 5600 50  0001 C CNN
@@
 $EndComp
 $Comp
-L GND #PWR09
+L GND #PWR18
 U 1 1 591E7037
 P 8300 2650
-F 0 "#PWR09" H 8300 2400 50  0001 C CNN
+F 0 "#PWR18" H 8300 2400 50  0001 C CNN
 F 1 "GND" H 8300 2500 50  0000 C CNN
 F 2 "" H 8300 2650 50  0001 C CNN
@@
 $EndComp
 $Comp
-L GND #PWR010
+L GND #PWR7
 U 1 1 591F4B78
 P 4200 3150
-F 0 "#PWR010" H 4200 2900 50  0001 C CNN
+F 0 "#PWR7" H 4200 2900 50  0001 C CNN
 F 1 "GND" H 4200 3000 50  0000 C CNN
 F 2 "" H 4200 3150 50  0001 C CNN
@@
 $EndComp
 $Comp
-L GND #PWR011
+L GND #PWR11
 U 1 1 591F4BD4
 P 4500 3150
-F 0 "#PWR011" H 4500 2900 50  0001 C CNN
+F 0 "#PWR11" H 4500 2900 50  0001 C CNN
 F 1 "GND" H 4500 3000 50  0000 C CNN
 F 2 "" H 4500 3150 50  0001 C CNN
@@
 $EndComp
 $Comp
-L GND #PWR012
+L GND #PWR12
 U 1 1 591F5A39
 P 4500 3350
-F 0 "#PWR012" H 4500 3100 50  0001 C CNN
+F 0 "#PWR12" H 4500 3100 50  0001 C CNN
 F 1 "GND" H 4500 3200 50  0000 C CNN
 F 2 "" H 4500 3350 50  0001 C CNN
@@
 $EndComp
 $Comp
-L GND #PWR013
+L GND #PWR8
 U 1 1 591F5A9B
 P 4200 3350
-F 0 "#PWR013" H 4200 3100 50  0001 C CNN
+F 0 "#PWR8" H 4200 3100 50  0001 C CNN
 F 1 "GND" H 4200 3200 50  0000 C CNN
 F 2 "" H 4200 3350 50  0001 C CNN
@@
 3V3
 $Comp
-L GND #PWR014
+L GND #PWR6
 U 1 1 591F843F
 P 4200 2150
-F 0 "#PWR014" H 4200 1900 50  0001 C CNN
+F 0 "#PWR6" H 4200 1900 50  0001 C CNN
 F 1 "GND" H 4200 2000 50  0000 C CNN
 F 2 "" H 4200 2150 50  0001 C CNN
@@
 $EndComp
 $Comp
-L GND #PWR?
+L GND #PWR9
 U 1 1 591FFF1B
 P 4200 3550
-F 0 "#PWR?" H 4200 3300 50  0001 C CNN
+F 0 "#PWR9" H 4200 3300 50  0001 C CNN
 F 1 "GND" H 4200 3400 50  0000 C CNN
 F 2 "" H 4200 3550 50  0001 C CNN
@@
 $EndComp
 $Comp
-L GND #PWR?
+L GND #PWR13
 U 1 1 591FFF8C
 P 4500 3550
-F 0 "#PWR?" H 4500 3300 50  0001 C CNN
+F 0 "#PWR13" H 4500 3300 50  0001 C CNN
 F 1 "GND" H 4500 3400 50  0000 C CNN
 F 2 "" H 4500 3550 50  0001 C CNN
@@
 	8950 2150 9050 2150
 Connection ~ 9000 2150
+Text GLabel 6500 2350 0    60   Input ~ 0
+3V3
+Text GLabel 9000 1850 1    60   Input ~ 0
+3V3
+$Comp
+L R RJ8
+U 1 1 59332C6E
+P 4350 3750
+F 0 "RJ8" V 4430 3750 50  0000 C CNN
+F 1 "0" V 4350 3750 50  0000 C CNN
+F 2 "Resistors_SMD:R_1206_HandSoldering" V 4280 3750 50  0001 C CNN
+F 3 "" H 4350 3750 50  0001 C CNN
+	1    4350 3750
+	0    1    1    0
+$EndComp
+$Comp
+L GND #PWR10
+U 1 1 59332CEF
+P 4200 3750
+F 0 "#PWR10" H 4200 3500 50  0001 C CNN
+F 1 "GND" H 4200 3600 50  0000 C CNN
+F 2 "" H 4200 3750 50  0001 C CNN
+F 3 "" H 4200 3750 50  0001 C CNN
+	1    4200 3750
+	0    1    1    0
+$EndComp
+$Comp
+L GND #PWR14
+U 1 1 59332D63
+P 4500 3750
+F 0 "#PWR14" H 4500 3500 50  0001 C CNN
+F 1 "GND" H 4500 3600 50  0000 C CNN
+F 2 "" H 4500 3750 50  0001 C CNN
+F 3 "" H 4500 3750 50  0001 C CNN
+	1    4500 3750
+	0    -1   -1   0
+$EndComp
 $EndSCHEMATC

Commit message: Mainboard changes
Parts:
- removed J7, J8: CONN_01X02, Pin_Headers:Pin_Header_Straight_1x02_Pitch2.54mm_SMD_Pin1Left, symbol CONN_01X02
- removed RJ6, RJ7: 0, Resistors_SMD:R_1206_HandSoldering, symbol R
- renumbered J9 to J7, RJ8 to RJ6
Connections:
- net 3V3: now also C3.1, C4.1, RJ3.1, RJ3.2, U1.2 (VO), U1.4 (VO), U3.3 (Vout); no longer J7.2 (P2)
- net GND: now also C1.2, C2.2, C3.2, C4.2, U1.1 (GND/ADJ), U3.2 (GND); no longer RJ3.1, RJ3.2
- net SD_D: now also RJ5.1
- net at D2.2 (A): now also J7.2 (P2)
Other:
- moved on the sheet: J7, R4, RJ6
Changed lines of the file:
@@
 3V3
 $Comp
-L GND #PWR1
+L GND #PWR01
 U 1 1 591DCE28
 P 2600 1750
-F 0 "#PWR1" H 2600 1500 50  0001 C CNN
+F 0 "#PWR01" H 2600 1500 50  0001 C CNN
 F 1 "GND" H 2600 1600 50  0000 C CNN
 F 2 "" H 2600 1750 50  0001 C CNN
@@
 SCK
 $Comp
-L GND #PWR2
+L GND #PWR02
 U 1 1 591DCE55
 P 2600 2450
-F 0 "#PWR2" H 2600 2200 50  0001 C CNN
+F 0 "#PWR02" H 2600 2200 50  0001 C CNN
 F 1 "GND" H 2600 2300 50  0000 C CNN
 F 2 "" H 2600 2450 50  0001 C CNN
@@
 $EndComp
 $Comp
-L GND #PWR4
+L GND #PWR03
 U 1 1 591DD033
 P 3650 1750
-F 0 "#PWR4" H 3650 1500 50  0001 C CNN
+F 0 "#PWR03" H 3650 1500 50  0001 C CNN
 F 1 "GND" H 3650 1600 50  0000 C CNN
 F 2 "" H 3650 1750 50  0001 C CNN
@@
 3V3
 $Comp
-L GND #PWR5
+L GND #PWR04
 U 1 1 591DD05E
 P 3650 2150
-F 0 "#PWR5" H 3650 1900 50  0001 C CNN
+F 0 "#PWR04" H 3650 1900 50  0001 C CNN
 F 1 "GND" H 3650 2000 50  0000 C CNN
 F 2 "" H 3650 2150 50  0001 C CNN
@@
 1wire
 $Comp
-L GND #PWR15
+L GND #PWR05
 U 1 1 591DD301
 P 5200 2850
-F 0 "#PWR15" H 5200 2600 50  0001 C CNN
+F 0 "#PWR05" H 5200 2600 50  0001 C CNN
 F 1 "GND" H 5200 2700 50  0000 C CNN
 F 2 "" H 5200 2850 50  0001 C CNN
@@
 MOSI
 $Comp
-L GND #PWR16
+L GND #PWR06
 U 1 1 591DDAB3
 P 6500 2250
-F 0 "#PWR16" H 6500 2000 50  0001 C CNN
+F 0 "#PWR06" H 6500 2000 50  0001 C CNN
 F 1 "GND" H 6500 2100 50  0000 C CNN
 F 2 "" H 6500 2250 50  0001 C CNN
@@
 SCK
 $Comp
-L GND #PWR17
+L GND #PWR07
 U 1 1 591DDB59
 P 6500 2550
-F 0 "#PWR17" H 6500 2300 50  0001 C CNN
+F 0 "#PWR07" H 6500 2300 50  0001 C CNN
 F 1 "GND" H 6500 2400 50  0000 C CNN
 F 2 "" H 6500 2550 50  0001 C CNN
@@
 L R R4
 U 1 1 591DDBFF
-P 9000 2000
-F 0 "R4" V 9080 2000 50  0000 C CNN
-F 1 "10k" V 9000 2000 50  0000 C CNN
-F 2 "Resistors_SMD:R_1206_HandSoldering" V 8930 2000 50  0001 C CNN
-F 3 "" H 9000 2000 50  0001 C CNN
-	1    9000 2000
-	1    0    0    -1
-$EndComp
-Text GLabel 9050 2150 2    60   Input ~ 0
+P 8700 2000
+F 0 "R4" V 8780 2000 50  0000 C CNN
+F 1 "10k" V 8700 2000 50  0000 C CNN
+F 2 "Resistors_SMD:R_1206_HandSoldering" V 8630 2000 50  0001 C CNN
+F 3 "" H 8700 2000 50  0001 C CNN
+	1    8700 2000
+	1    0    0    -1
+$EndComp
+Text GLabel 8750 2150 2    60   Input ~ 0
 SD_D
 $Comp
@@
 3V3
 $Comp
-L GND #PWR3
+L GND #PWR08
 U 1 1 591DF8F9
 P 3300 5600
-F 0 "#PWR3" H 3300 5350 50  0001 C CNN
+F 0 "#PWR08" H 3300 5350 50  0001 C CNN
 F 1 "GND" H 3300 5450 50  0000 C CNN
 F 2 "" H 3300 5600 50  0001 C CNN
@@
 $EndComp
 $Comp
-L CONN_01X02 J7
-U 1 1 591E38B8
-P 4700 4500
-F 0 "J7" H 4700 4650 50  0000 C CNN
-F 1 "CONN_01X02" V 4800 4500 50  0000 C CNN
-F 2 "Pin_Headers:Pin_Header_Straight_1x02_Pitch2.54mm_SMD_Pin1Left" H 4700 4500 50  0001 C CNN
-F 3 "" H 4700 4500 50  0001 C CNN
-	1    4700 4500
-	-1   0    0    1
-$EndComp
-$Comp
 L CONN_01X02 J6
 U 1 1 591E39F7
@@
 $EndComp
 $Comp
-L GND #PWR18
+L GND #PWR09
 U 1 1 591E7037
 P 8300 2650
-F 0 "#PWR18" H 8300 2400 50  0001 C CNN
+F 0 "#PWR09" H 8300 2400 50  0001 C CNN
 F 1 "GND" H 8300 2500 50  0000 C CNN
 F 2 "" H 8300 2650 50  0001 C CNN
@@
 $EndComp
 $Comp
-L GND #PWR7
-U 1 1 591F4B78
-P 4200 3150
-F 0 "#PWR7" H 4200 2900 50  0001 C CNN
-F 1 "GND" H 4200 3000 50  0000 C CNN
-F 2 "" H 4200 3150 50  0001 C CNN
-F 3 "" H 4200 3150 50  0001 C CNN
-	1    4200 3150
-	0    1    1    0
-$EndComp
-$Comp
-L GND #PWR11
-U 1 1 591F4BD4
-P 4500 3150
-F 0 "#PWR11" H 4500 2900 50  0001 C CNN
-F 1 "GND" H 4500 3000 50  0000 C CNN
-F 2 "" H 4500 3150 50  0001 C CNN
-F 3 "" H 4500 3150 50  0001 C CNN
-	1    4500 3150
-	0    -1   -1   0
-$EndComp
-$Comp
 L R RJ3
 U 1 1 591F4C30
@@
 $EndComp
 $Comp
-L GND #PWR12
+L GND #PWR010
 U 1 1 591F5A39
 P 4500 3350
-F 0 "#PWR12" H 4500 3100 50  0001 C CNN
+F 0 "#PWR010" H 4500 3100 50  0001 C CNN
 F 1 "GND" H 4500 3200 50  0000 C CNN
 F 2 "" H 4500 3350 50  0001 C CNN
@@
 $EndComp
 $Comp
-L GND #PWR8
+L GND #PWR011
 U 1 1 591F5A9B
 P 4200 3350
-F 0 "#PWR8" H 4200 3100 50  0001 C CNN
+F 0 "#PWR011" H 4200 3100 50  0001 C CNN
 F 1 "GND" H 4200 3200 50  0000 C CNN
 F 2 "" H 4200 3350 50  0001 C CNN
@@
 $EndComp
 $Comp
-L CONN_01X02 J8
-U 1 1 591F7076
-P 7150 5250
-F 0 "J8" H 7150 5400 50  0000 C CNN
-F 1 "CONN_01X02" V 7250 5250 50  0000 C CNN
-F 2 "Pin_Headers:Pin_Header_Straight_1x02_Pitch2.54mm_SMD_Pin1Left" H 7150 5250 50  0001 C CNN
-F 3 "" H 7150 5250 50  0001 C CNN
-	1    7150 5250
-	1    0    0    1
-$EndComp
-$Comp
-L CONN_01X02 J9
+L CONN_01X02 J7
 U 1 1 591F80FA
-P 4400 2100
-F 0 "J9" H 4400 2250 50  0000 C CNN
-F 1 "CONN_01X02" V 4500 2100 50  0000 C CNN
-F 2 "Pin_Headers:Pin_Header_Straight_1x02_Pitch2.54mm_SMD_Pin1Left" H 4400 2100 50  0001 C CNN
-F 3 "" H 4400 2100 50  0001 C CNN
-	1    4400 2100
-	1    0    0    1
-$EndComp
-Text GLabel 4200 2050 0    60   Input ~ 0
-3V3
-$Comp
-L GND #PWR6
-U 1 1 591F843F
-P 4200 2150
-F 0 "#PWR6" H 4200 1900 50  0001 C CNN
-F 1 "GND" H 4200 2000 50  0000 C CNN
-F 2 "" H 4200 2150 50  0001 C CNN
-F 3 "" H 4200 2150 50  0001 C CNN
-	1    4200 2150
-	1    0    0    -1
-$EndComp
-$Comp
-L R RJ6
-U 1 1 591F890C
-P 8800 2150
-F 0 "RJ6" V 8880 2150 50  0000 C CNN
-F 1 "0" V 8800 2150 50  0000 C CNN
-F 2 "Resistors_SMD:R_1206_HandSoldering" V 8730 2150 50  0001 C CNN
-F 3 "" H 8800 2150 50  0001 C CNN
-	1    8800 2150
-	0    1    1    0
+P 4700 4500
+F 0 "J7" H 4700 4650 50  0000 C CNN
+F 1 "CONN_01X02" V 4800 4500 50  0000 C CNN
+F 2 "Pin_Headers:Pin_Header_Straight_1x02_Pitch2.54mm_SMD_Pin1Left" H 4700 4500 50  0001 C CNN
+F 3 "" H 4700 4500 50  0001 C CNN
+	1    4700 4500
+	-1   0    0    1
 $EndComp
 $Comp
@@
 Wire Wire Line
 	4900 4550 4900 5500
-Wire Wire Line
-	4900 5500 6950 5500
 Connection ~ 5700 4450
 Wire Wire Line
@@
 Wire Wire Line
 	2150 2300 2450 2300
-Wire Wire Line
-	6950 5500 6950 5300
 Connection ~ 6800 5500
 Wire Wire Line
@@
 Connection ~ 6250 5500
 Wire Wire Line
-	8600 2150 8650 2150
-$Comp
-L R RJ7
-U 1 1 591FFE8B
+	8600 2150 8750 2150
+Connection ~ 8700 2150
+Text GLabel 6500 2350 0    60   Input ~ 0
+3V3
+Text GLabel 8700 1850 1    60   Input ~ 0
+3V3
+$Comp
+L R RJ6
+U 1 1 59332C6E
 P 4350 3550
-F 0 "RJ7" V 4430 3550 50  0000 C CNN
+F 0 "RJ6" V 4430 3550 50  0000 C CNN
 F 1 "0" V 4350 3550 50  0000 C CNN
 F 2 "Resistors_SMD:R_1206_HandSoldering" V 4280 3550 50  0001 C CNN
@@
 $EndComp
 $Comp
-L GND #PWR9
-U 1 1 591FFF1B
+L GND #PWR014
+U 1 1 59332CEF
 P 4200 3550
-F 0 "#PWR9" H 4200 3300 50  0001 C CNN
+F 0 "#PWR014" H 4200 3300 50  0001 C CNN
 F 1 "GND" H 4200 3400 50  0000 C CNN
 F 2 "" H 4200 3550 50  0001 C CNN
@@
 $EndComp
 $Comp
-L GND #PWR13
-U 1 1 591FFF8C
+L GND #PWR015
+U 1 1 59332D63
 P 4500 3550
-F 0 "#PWR13" H 4500 3300 50  0001 C CNN
+F 0 "#PWR015" H 4500 3300 50  0001 C CNN
 F 1 "GND" H 4500 3400 50  0000 C CNN
 F 2 "" H 4500 3550 50  0001 C CNN
@@
 	0    -1   -1   0
 $EndComp
-Wire Wire Line
-	8950 2150 9050 2150
-Connection ~ 9000 2150
-Text GLabel 6500 2350 0    60   Input ~ 0
-3V3
-Text GLabel 9000 1850 1    60   Input ~ 0
-3V3
-$Comp
-L R RJ8
-U 1 1 59332C6E
-P 4350 3750
-F 0 "RJ8" V 4430 3750 50  0000 C CNN
-F 1 "0" V 4350 3750 50  0000 C CNN
-F 2 "Resistors_SMD:R_1206_HandSoldering" V 4280 3750 50  0001 C CNN
-F 3 "" H 4350 3750 50  0001 C CNN
-	1    4350 3750
-	0    1    1    0
-$EndComp
-$Comp
-L GND #PWR10
-U 1 1 59332CEF
-P 4200 3750
-F 0 "#PWR10" H 4200 3500 50  0001 C CNN
-F 1 "GND" H 4200 3600 50  0000 C CNN
-F 2 "" H 4200 3750 50  0001 C CNN
-F 3 "" H 4200 3750 50  0001 C CNN
-	1    4200 3750
-	0    1    1    0
-$EndComp
-$Comp
-L GND #PWR14
-U 1 1 59332D63
-P 4500 3750
-F 0 "#PWR14" H 4500 3500 50  0001 C CNN
-F 1 "GND" H 4500 3600 50  0000 C CNN
-F 2 "" H 4500 3750 50  0001 C CNN
-F 3 "" H 4500 3750 50  0001 C CNN
-	1    4500 3750
-	0    -1   -1   0
-$EndComp
+Text GLabel 6950 5200 2    60   Input ~ 0
+3V3
+$Comp
+L GND #PWR016
+U 1 1 594541DB
+P 7050 5500
+F 0 "#PWR016" H 7050 5250 50  0001 C CNN
+F 1 "GND" H 7050 5350 50  0000 C CNN
+F 2 "" H 7050 5500 50  0001 C CNN
+F 3 "" H 7050 5500 50  0001 C CNN
+	1    7050 5500
+	1    0    0    -1
+$EndComp
+Wire Wire Line
+	4900 5500 7050 5500
+Text GLabel 4500 3150 2    60   Input ~ 0
+3V3
+Text GLabel 4200 3150 0    60   Input ~ 0
+3V3
 $EndSCHEMATC
