File: PCF8563_PCB/Mainboard1.1_LM1117/Mainboard1.1_LM1117.sch (KiCad schematic (older format))
At the start: 30 parts, among them J1 CONN_01X03, J2 CONN_01X15, J3 CONN_01X15, J4 SD_Card, J5 CONN_01X03, J6 CONN_01X02, J7 CONN_01X02, U1 LM1117-3.3, U2 PCF8563, Y1 Crystal

Commit message: SettingsGenerator update
Added validating addresses in SettingsGenerator
Modified LM1117 board (SOT instead of DPAK voltage stabiliser)
Something I forgot
Parts:
- U1: footprint TO_SOT_Packages_SMD:TO-252-2 -> TO_SOT_Packages_SMD:SOT-223-3Lead_TabPin2
Changed lines of the file:
@@
 LIBS:contrib
 LIBS:valves
-LIBS:Mainboard_1.1-cache
+LIBS:Mainboard1.1_LM1117-cache
 EELAYER 25 0
 EELAYER END
@@
 F 0 "U1" H 6100 4950 50  0000 C CNN
 F 1 "LM1117-3.3" H 6000 5450 50  0000 C CNN
-F 2 "TO_SOT_Packages_SMD:TO-252-2" H 6000 5200 50  0001 C CNN
+F 2 "TO_SOT_Packages_SMD:SOT-223-3Lead_TabPin2" H 6000 5200 50  0001 C CNN
 F 3 "" H 6000 5200 50  0001 C CNN
 	1    6000 5200
@@
 $EndComp
 $Comp
-L GND #PWR014
+L GND #PWR012
 U 1 1 59332CEF
 P 4200 3550
-F 0 "#PWR014" H 4200 3300 50  0001 C CNN
+F 0 "#PWR012" H 4200 3300 50  0001 C CNN
 F 1 "GND" H 4200 3400 50  0000 C CNN
 F 2 "" H 4200 3550 50  0001 C CNN
@@
 $EndComp
 $Comp
-L GND #PWR015
+L GND #PWR013
 U 1 1 59332D63
 P 4500 3550
-F 0 "#PWR015" H 4500 3300 50  0001 C CNN
+F 0 "#PWR013" H 4500 3300 50  0001 C CNN
 F 1 "GND" H 4500 3400 50  0000 C CNN
 F 2 "" H 4500 3550 50  0001 C CNN
@@
 3V3
 $Comp
-L GND #PWR016
+L GND #PWR014
 U 1 1 594541DB
 P 7050 5500
-F 0 "#PWR016" H 7050 5250 50  0001 C CNN
+F 0 "#PWR014" H 7050 5250 50  0001 C CNN
 F 1 "GND" H 7050 5350 50  0000 C CNN
 F 2 "" H 7050 5500 50  0001 C CNN
