File: Temperature-Station_PCF8563_JSON/PCF8563_PCB/Mainboard1.1_LM1117/Mainboard1.1_LM1117.sch (KiCad schematic (older format))
At the start: 30 parts, among them J1 CONN_01X03, J2 CONN_01X15, J3 CONN_01X15, J4 SD_Card, J5 CONN_01X03, J6 CONN_01X02, J7 CONN_01X02, U1 LM1117-3.3, U2 PCF8563, Y1 Crystal

Commit message: Updates
Updated both versions
Added online updater
Minor cosmetic changes
Saving DHCP settings restored
Added authentication (still no HTTPS/TLS/SSL tho)
Moved as many Strings as possible to Flash memory to free RAM

Czas library:
Optimized for porting between DS3231 and PCF8563 versions.
Parts:
- added RJ7, RJ8: 0, Resistors_SMD:R_1206_HandSoldering, symbol R
- J7: footprint Pin_Headers:Pin_Header_Straight_1x02_Pitch2.54mm_SMD_Pin1Left -> Socket_Strips:Socket_Strip_Angled_1x02_Pitch2.54mm
- U1: symbol LM1117-3.3 -> LM1117-3.3-RESCUE-Mainboard1.1_LM1117
Connections:
- net 3V3: now also RJ7.1, RJ7.2
- net GND: now also J7.2 (P2), RJ8.1, RJ8.2; no longer J7.1 (P1)
- net at D2.2 (A): now also J7.1 (P1); no longer J7.2 (P2)
Other:
- moved on the sheet: RJ2, RJ3, RJ4, RJ6
Changed lines of the file:
@@
 EESchema Schematic File Version 2
+LIBS:Mainboard1.1_LM1117-rescue
 LIBS:power
 LIBS:device
@@
 LIBS:valves
 LIBS:Mainboard1.1_LM1117-cache
-EELAYER 25 0
+EELAYER 26 0
 EELAYER END
 $Descr A4 11693 8268
@@
 $EndComp
 $Comp
-L LM1117-3.3 U1
+L LM1117-3.3-RESCUE-Mainboard1.1_LM1117 U1
 U 1 1 591E00AF
 P 6000 5200
@@
 	0    1    1    0
 $EndComp
-Text GLabel 4200 2950 0    60   Input ~ 0
-3V3
-Text GLabel 4500 2950 2    60   Input ~ 0
+Text GLabel 4250 3000 0    60   Input ~ 0
+3V3
+Text GLabel 4550 3000 2    60   Input ~ 0
 3V3
 $Comp
 L R RJ2
 U 1 1 591F46BE
-P 4350 2950
-F 0 "RJ2" V 4430 2950 50  0000 C CNN
-F 1 "0" V 4350 2950 50  0000 C CNN
-F 2 "Resistors_SMD:R_1206_HandSoldering" V 4280 2950 50  0001 C CNN
-F 3 "" H 4350 2950 50  0001 C CNN
-	1    4350 2950
+P 4400 3000
+F 0 "RJ2" V 4480 3000 50  0000 C CNN
+F 1 "0" V 4400 3000 50  0000 C CNN
+F 2 "Resistors_SMD:R_1206_HandSoldering" V 4330 3000 50  0001 C CNN
+F 3 "" H 4400 3000 50  0001 C CNN
+	1    4400 3000
 	0    1    1    0
 $EndComp
@@
 L R RJ3
 U 1 1 591F4C30
-P 4350 3150
-F 0 "RJ3" V 4430 3150 50  0000 C CNN
-F 1 "0" V 4350 3150 50  0000 C CNN
-F 2 "Resistors_SMD:R_1206_HandSoldering" V 4280 3150 50  0001 C CNN
-F 3 "" H 4350 3150 50  0001 C CNN
-	1    4350 3150
+P 4400 3200
+F 0 "RJ3" V 4480 3200 50  0000 C CNN
+F 1 "0" V 4400 3200 50  0000 C CNN
+F 2 "Resistors_SMD:R_1206_HandSoldering" V 4330 3200 50  0001 C CNN
+F 3 "" H 4400 3200 50  0001 C CNN
+	1    4400 3200
 	0    1    1    0
 $EndComp
@@
 L R RJ4
 U 1 1 591F59BA
-P 4350 3350
-F 0 "RJ4" V 4430 3350 50  0000 C CNN
-F 1 "0" V 4350 3350 50  0000 C CNN
-F 2 "Resistors_SMD:R_1206_HandSoldering" V 4280 3350 50  0001 C CNN
-F 3 "" H 4350 3350 50  0001 C CNN
-	1    4350 3350
+P 4400 3600
+F 0 "RJ4" V 4480 3600 50  0000 C CNN
+F 1 "0" V 4400 3600 50  0000 C CNN
+F 2 "Resistors_SMD:R_1206_HandSoldering" V 4330 3600 50  0001 C CNN
+F 3 "" H 4400 3600 50  0001 C CNN
+	1    4400 3600
 	0    1    1    0
 $EndComp
@@
 L GND #PWR010
 U 1 1 591F5A39
-P 4500 3350
-F 0 "#PWR010" H 4500 3100 50  0001 C CNN
-F 1 "GND" H 4500 3200 50  0000 C CNN
-F 2 "" H 4500 3350 50  0001 C CNN
-F 3 "" H 4500 3350 50  0001 C CNN
-	1    4500 3350
+P 4550 3600
+F 0 "#PWR010" H 4550 3350 50  0001 C CNN
+F 1 "GND" H 4550 3450 50  0000 C CNN
+F 2 "" H 4550 3600 50  0001 C CNN
+F 3 "" H 4550 3600 50  0001 C CNN
+	1    4550 3600
 	0    -1   -1   0
 $EndComp
@@
 L GND #PWR011
 U 1 1 591F5A9B
-P 4200 3350
-F 0 "#PWR011" H 4200 3100 50  0001 C CNN
-F 1 "GND" H 4200 3200 50  0000 C CNN
-F 2 "" H 4200 3350 50  0001 C CNN
-F 3 "" H 4200 3350 50  0001 C CNN
-	1    4200 3350
+P 4250 3600
+F 0 "#PWR011" H 4250 3350 50  0001 C CNN
+F 1 "GND" H 4250 3450 50  0000 C CNN
+F 2 "" H 4250 3600 50  0001 C CNN
+F 3 "" H 4250 3600 50  0001 C CNN
+	1    4250 3600
 	0    1    1    0
 $EndComp
@@
 F 0 "J7" H 4700 4650 50  0000 C CNN
 F 1 "CONN_01X02" V 4800 4500 50  0000 C CNN
-F 2 "Pin_Headers:Pin_Header_Straight_1x02_Pitch2.54mm_SMD_Pin1Left" H 4700 4500 50  0001 C CNN
+F 2 "Socket_Strips:Socket_Strip_Angled_1x02_Pitch2.54mm" H 4700 4500 50  0001 C CNN
 F 3 "" H 4700 4500 50  0001 C CNN
 	1    4700 4500
-	-1   0    0    1
+	-1   0    0    -1
 $EndComp
 $Comp
@@
 L R RJ6
 U 1 1 59332C6E
-P 4350 3550
-F 0 "RJ6" V 4430 3550 50  0000 C CNN
-F 1 "0" V 4350 3550 50  0000 C CNN
-F 2 "Resistors_SMD:R_1206_HandSoldering" V 4280 3550 50  0001 C CNN
-F 3 "" H 4350 3550 50  0001 C CNN
-	1    4350 3550
+P 4400 3800
+F 0 "RJ6" V 4480 3800 50  0000 C CNN
+F 1 "0" V 4400 3800 50  0000 C CNN
+F 2 "Resistors_SMD:R_1206_HandSoldering" V 4330 3800 50  0001 C CNN
+F 3 "" H 4400 3800 50  0001 C CNN
+	1    4400 3800
 	0    1    1    0
 $EndComp
@@
 L GND #PWR012
 U 1 1 59332CEF
-P 4200 3550
-F 0 "#PWR012" H 4200 3300 50  0001 C CNN
-F 1 "GND" H 4200 3400 50  0000 C CNN
-F 2 "" H 4200 3550 50  0001 C CNN
-F 3 "" H 4200 3550 50  0001 C CNN
-	1    4200 3550
+P 4250 3800
+F 0 "#PWR012" H 4250 3550 50  0001 C CNN
+F 1 "GND" H 4250 3650 50  0000 C CNN
+F 2 "" H 4250 3800 50  0001 C CNN
+F 3 "" H 4250 3800 50  0001 C CNN
+	1    4250 3800
 	0    1    1    0
 $EndComp
@@
 L GND #PWR013
 U 1 1 59332D63
-P 4500 3550
-F 0 "#PWR013" H 4500 3300 50  0001 C CNN
-F 1 "GND" H 4500 3400 50  0000 C CNN
-F 2 "" H 4500 3550 50  0001 C CNN
-F 3 "" H 4500 3550 50  0001 C CNN
-	1    4500 3550
+P 4550 3800
+F 0 "#PWR013" H 4550 3550 50  0001 C CNN
+F 1 "GND" H 4550 3650 50  0000 C CNN
+F 2 "" H 4550 3800 50  0001 C CNN
+F 3 "" H 4550 3800 50  0001 C CNN
+	1    4550 3800
 	0    -1   -1   0
 $EndComp
@@
 Wire Wire Line
 	4900 5500 7050 5500
-Text GLabel 4500 3150 2    60   Input ~ 0
-3V3
-Text GLabel 4200 3150 0    60   Input ~ 0
+Text GLabel 4550 3200 2    60   Input ~ 0
+3V3
+Text GLabel 4250 3200 0    60   Input ~ 0
 3V3
 Connection ~ 6000 5500
+$Comp
+L R RJ8
+U 1 1 59F500C9
+P 4400 4000
+F 0 "RJ8" V 4480 4000 50  0000 C CNN
+F 1 "0" V 4400 4000 50  0000 C CNN
+F 2 "Resistors_SMD:R_1206_HandSoldering" V 4330 4000 50  0001 C CNN
+F 3 "" H 4400 4000 50  0001 C CNN
+	1    4400 4000
+	0    1    1    0
+$EndComp
+$Comp
+L GND #PWR015
+U 1 1 59F500CF
+P 4250 4000
+F 0 "#PWR015" H 4250 3750 50  0001 C CNN
+F 1 "GND" H 4250 3850 50  0000 C CNN
+F 2 "" H 4250 4000 50  0001 C CNN
+F 3 "" H 4250 4000 50  0001 C CNN
+	1    4250 4000
+	0    1    1    0
+$EndComp
+$Comp
+L GND #PWR016
+U 1 1 59F500D5
+P 4550 4000
+F 0 "#PWR016" H 4550 3750 50  0001 C CNN
+F 1 "GND" H 4550 3850 50  0000 C CNN
+F 2 "" H 4550 4000 50  0001 C CNN
+F 3 "" H 4550 4000 50  0001 C CNN
+	1    4550 4000
+	0    -1   -1   0
+$EndComp
+$Comp
+L R RJ7
+U 1 1 59F50312
+P 4400 3400
+F 0 "RJ7" V 4480 3400 50  0000 C CNN
+F 1 "0" V 4400 3400 50  0000 C CNN
+F 2 "Resistors_SMD:R_1206_HandSoldering" V 4330 3400 50  0001 C CNN
+F 3 "" H 4400 3400 50  0001 C CNN
+	1    4400 3400
+	0    1    1    0
+$EndComp
+Text GLabel 4550 3400 2    60   Input ~ 0
+3V3
+Text GLabel 4250 3400 0    60   Input ~ 0
+3V3
 $EndSCHEMATC
