File: Temperature-Station_PCF8563_JSON/PCF8563_PCB/Mainboard2.0_LM1117_SERIAL/Mainboard2.0_LM1117.sch (KiCad schematic (older format))
At the start: 32 parts, among them J1 CONN_01X03, J2 CONN_01X03, J4 SD_Card, J5 CONN_01X03, J6 CONN_01X02, J7 CONN_01X02, SW1 RESET, SW2 FLASH, U1 LM1117-3.3, U2 PCF8563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

Commit message: Updates
Updated both versions
Added online updater
Minor cosmetic changes
Saving DHCP settings restored
Added authentication (still no HTTPS/TLS/SSL tho)
Moved as many Strings as possible to Flash memory to free RAM

Czas library:
Optimized for porting between DS3231 and PCF8563 versions.
Parts:
- SW1, SW2: symbol SW_DIP_x01 -> SW_DIP_x01-RESCUE-Mainboard2.0_LM1117
Changed lines of the file:
@@
 LIBS:contrib
 LIBS:valves
-LIBS:ESP8266
 LIBS:74xgxx
 LIBS:ac-dc
@@
 LIBS:ftdi
 LIBS:gennum
-LIBS:graphic
 LIBS:graphic_symbols
 LIBS:hc11
@@
 LIBS:leds
 LIBS:LEM
-LIBS:logo
 LIBS:maxim
 LIBS:mechanical
@@
 RESET
 $Comp
-L SW_DIP_x01 SW1
+L SW_DIP_x01-RESCUE-Mainboard2.0_LM1117 SW1
 U 1 1 5962EC4D
 P 3550 4600
@@
 	8650 3150 8650 3800
 $Comp
-L SW_DIP_x01 SW2
+L SW_DIP_x01-RESCUE-Mainboard2.0_LM1117 SW2
 U 1 1 596B81BC
 P 2800 4600
