File: Temperature-Station_PCF8563/PCF8563_PCB/RJ45_I2C_1.0/RJ45_I2C_1.0.sch (KiCad schematic (older format))
At the start: 28 parts, among them J0 MHRJJ66NFRA, J1 MHRJJ66NFRA, J2 MHRJJ66NFRA, J3 MHRJJ66NFRA, J4 MHRJJ66NFRA, J5 MHRJJ66NFRA, J6 MHRJJ66NFRA, J7 MHRJJ66NFRA, J8 Out, J9 Prog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

Commit message: Updated boards and sketches
Boards:
Sandwich-like layout so you can connect directly do DHT sensors or use i2c expansion (8 slots).
Boards support 1wire, DHT11/21/22 sensors and require custom wiring.
Reduced size of boards

Sketch:
Hermetized settings (no way to read passwords)
Used settingsHandler to hold every field that will have to be saved
Fixed AP launch in PCF8563
Rolled back Pinger library due to readability issues.
WIP: Use external memory only for emergency sensor file and permanently for readings
TESTING: Update via curl
TESTING: Set time and date via webpage
WIP: Change settings via webpage
WIP: Change login credentials via webpage
Documentation: coming soon
Parts:
- removed J0, J1, J2, J3, J4, J5, J6, J7: MHRJJ66NFRA, MHRJJ66NFRA:MHRJJ66NFRA, symbol MHRJJ66NFRA:MHRJJ66NFRA
- removed R1, R2, R3, R4, R5, R6, R7, R8: 4k7, Resistor_SMD:R_1206_3216Metric, symbol Device:R
- removed R10, R11, R12, R13, R15, R16, R17, R9: 10k, Resistor_SMD:R_1206_3216Metric, symbol Device:R
- added J1: Conn_01x12, Connector_PinSocket_2.54mm:PinSocket_1x12_P2.54mm_Vertical, symbol Connector_Generic:Conn_01x12
- renumbered J8 to J2, J9 to J3, R14 to R1
Connections:
- net labels added: Vin
- wire segments 101 -> 11
Other:
- moved on the sheet: U1

Commit message: Muxtemp update
1wire option added
Working in bypass or local mode (if master can use 1wire it will NOT use 1wire devices)
Example shows more info
Parts:
- added JP1: bypass1Wire, Resistor_SMD:R_0805_2012Metric_Pad1.15x1.50mm_HandSolder, symbol Device:Jumper_NO_Small
Connections:
- wire segments 11 -> 12
Changed lines of the file:
@@
 Text GLabel 3200 3750 2    50   Input ~ 0
 SDA
-$Comp
-L Connector_Generic:Conn_01x05 J2
-U 1 1 5ADE7775
-P 5150 3400
-F 0 "J2" H 5230 3442 50  0000 L CNN
-F 1 "Out" H 5230 3351 50  0000 L CNN
-F 2 "Connector_PinHeader_2.54mm:PinHeader_1x05_P2.54mm_Vertical" H 5150 3400 50  0001 C CNN
-F 3 "~" H 5150 3400 50  0001 C CNN
-	1    5150 3400
-	1    0    0    -1
-$EndComp
 Text GLabel 4950 3500 0    50   Input ~ 0
 SDA
 Text GLabel 4950 3400 0    50   Input ~ 0
 SCL
-Text GLabel 4950 3600 0    50   Input ~ 0
-1wire
 Text GLabel 4950 3300 0    50   Input ~ 0
 3V3
@@
 Wire Wire Line
 	4650 3200 4950 3200
-Text GLabel 3200 3650 2    50   Input ~ 0
-1wire
 $Comp
 L Connector_Generic:Conn_01x12 J1
@@
 	1    0    0    -1
 $EndComp
+$Comp
+L Device:Jumper_NO_Small JP1
+U 1 1 5B11B726
+P 3300 3650
+F 0 "JP1" H 3450 3850 50  0000 C CNN
+F 1 "bypass1Wire" H 3450 3750 50  0000 C CNN
+F 2 "Resistor_SMD:R_0805_2012Metric_Pad1.15x1.50mm_HandSolder" H 3300 3650 50  0001 C CNN
+F 3 "~" H 3300 3650 50  0001 C CNN
+	1    3300 3650
+	1    0    0    -1
+$EndComp
+$Comp
+L power:GND #PWR0101
+U 1 1 5B11B9A1
+P 3600 3650
+F 0 "#PWR0101" H 3600 3400 50  0001 C CNN
+F 1 "GND" H 3605 3477 50  0000 C CNN
+F 2 "" H 3600 3650 50  0001 C CNN
+F 3 "" H 3600 3650 50  0001 C CNN
+	1    3600 3650
+	1    0    0    -1
+$EndComp
+Wire Wire Line
+	3400 3650 3600 3650
+Text GLabel 4950 3600 0    50   Input ~ 0
+1wire
+$Comp
+L Connector_Generic:Conn_01x05 J2
+U 1 1 5ADE7775
+P 5150 3400
+F 0 "J2" H 5230 3442 50  0000 L CNN
+F 1 "Out" H 5230 3351 50  0000 L CNN
+F 2 "Connector_PinHeader_2.54mm:PinHeader_1x05_P2.54mm_Vertical" H 5150 3400 50  0001 C CNN
+F 3 "~" H 5150 3400 50  0001 C CNN
+	1    5150 3400
+	1    0    0    -1
+$EndComp
