File: Temperature-Station_PCF8563/PCF8563_PCB/RJ45_Breakout/RJ45_Breakout.sch (KiCad schematic (older format))
At the start: 31 parts, among them J1 MHRJJ66NFRA, J2 MHRJJ66NFRA, J3 MHRJJ66NFRA, J4 MHRJJ66NFRA, J5 MHRJJ66NFRA, J6 MHRJJ66NFRA, J7 MHRJJ66NFRA, J8 MHRJJ66NFRA, J9 Flex, U1 LM1117-3.3

Commit message: Cleaned boards up
Merged RJ45_I2C with RJ45_Breakout into one schematic
Added fully-integrated Muxtemp board
Started working on Mainboard+Muxtemp board

Settings page (html) is now functional. Backend WIP.

SettingsHandler(PCF8563) is now cleaned up a bit, added optional define to include debug interface
Added option to configure OTA updater as well as WebUpdater
SettingsHandler(Slave): see above
Parts:
- added J10: Prog, Connector_PinSocket_2.54mm:PinSocket_1x04_P2.54mm_Vertical, symbol Connector_Generic:Conn_01x04
- added J11: Out, Connector_PinHeader_2.54mm:PinHeader_1x05_P2.54mm_Horizontal, symbol Connector_Generic:Conn_01x05
- added J9: Conn_01x12, Connector_PinSocket_2.54mm:PinSocket_1x12_P2.54mm_Vertical, symbol Connector_Generic:Conn_01x12
- added JP1: bypass1Wire, Resistor_SMD:R_0805_2012Metric_Pad1.15x1.50mm_HandSolder, symbol Device:Jumper_NO_Small
- added R9: 10k, Resistor_SMD:R_1206_3216Metric, symbol Device:R
- added U2: ATmega328-PU, Package_DIP:DIP-28_W7.62mm, symbol MCU_Microchip_ATmega:ATmega328-PU
- J12: renamed from J9; footprint Connector_PinHeader_2.54mm:PinHeader_1x16_P2.54mm_Vertical -> Connector_PinHeader_2.54mm:PinHeader_1x12_P2.54mm_Vertical
- renumbered R9 to R10, R10 to R11, R11 to R12, R12 to R13, R13 to R14, R14 to R15, R15 to R16, R16 to R17
Connections:
- net labels added: SCL, SDA
- wire segments 96 -> 108
Other:
- moved on the sheet: U1
