File: Boards/Mainboard_Final/Mainboard_Final.sch (KiCad schematic (older format))
At the start: 71 parts

Commit message: Optimizations and updates
PCF8563:
Added non-address version (sensor dosen't override port name)
Finished settings
Index and settings are stored in sketch, not SD-card
Minor optimization (migrate to const char* instead of string)
Temporarily disabled remote devices
Bigger buffer for sensors file
Added option to change port names in /sensors
Removed file manipulation from HTTPserver

Muxtemp:
Added hardware lock check
Minor changes

Boards:
Moved to different folder

SettingsHandler:
Set up config file during object initialization
Minor optimization
Added printConfig and printConfigFile (debug mode only)

I2C Expander:
Changed DS18B20 type to 40
Addded hardware lock
Changed lines of the file:
@@
 EESchema Schematic File Version 4
-LIBS:Mainboard_4.0-cache
-LIBS:RJ45_I2C_2.0-cache
+LIBS:Mainboard_Final-cache
 EELAYER 26 0
 EELAYER END
@@
 L Device:R R?
 U 1 1 5ACB2116
-P 2800 3200
-F 0 "R?" V 2800 3200 50  0000 C CNN
-F 1 "4k7" V 2800 3750 50  0000 C CNN
-F 2 "" V 2730 3200 50  0001 C CNN
-F 3 "~" H 2800 3200 50  0001 C CNN
-	1    2800 3200
+P 2800 3300
+F 0 "R?" V 2800 3300 50  0000 C CNN
+F 1 "4k7" V 2800 3850 50  0000 C CNN
+F 2 "" V 2730 3300 50  0001 C CNN
+F 3 "~" H 2800 3300 50  0001 C CNN
+	1    2800 3300
 	0    -1   -1   0
 $EndComp
@@
 $EndComp
 Wire Wire Line
-	2600 3250 2950 3250
-Wire Wire Line
-	2950 3250 2950 3200
-Wire Wire Line
 	2600 2950 2650 2950
 $Comp
@@
 	1750 3500 1850 3500
 Connection ~ 1750 3500
-Connection ~ 2950 3200
-Wire Wire Line
-	2650 3100 2650 3200
-Connection ~ 2650 3100
 Connection ~ 2950 3100
 Wire Wire Line
@@
 L Device:R R?
 U 1 1 5B08A8A2
-P 4850 6550
-F 0 "R?" V 4850 6900 50  0000 C CNN
-F 1 "33k" V 4850 7050 50  0000 C CNN
-F 2 "" V 4780 6550 50  0001 C CNN
-F 3 "~" H 4850 6550 50  0001 C CNN
-	1    4850 6550
+P 4400 6000
+F 0 "R?" V 4400 6350 50  0000 C CNN
+F 1 "33k" V 4400 6500 50  0000 C CNN
+F 2 "" V 4330 6000 50  0001 C CNN
+F 3 "~" H 4400 6000 50  0001 C CNN
+	1    4400 6000
 	0    -1   -1   0
 $EndComp
@@
 L power:GND #PWR?
 U 1 1 5B08E015
-P 4700 7300
-F 0 "#PWR?" H 4700 7050 50  0001 C CNN
-F 1 "GND" H 4705 7127 50  0000 C CNN
-F 2 "" H 4700 7300 50  0001 C CNN
-F 3 "" H 4700 7300 50  0001 C CNN
-	1    4700 7300
+P 4250 6750
+F 0 "#PWR?" H 4250 6500 50  0001 C CNN
+F 1 "GND" H 4255 6577 50  0000 C CNN
+F 2 "" H 4250 6750 50  0001 C CNN
+F 3 "" H 4250 6750 50  0001 C CNN
+	1    4250 6750
 	1    0    0    -1
 $EndComp
@@
 L Device:R R?
 U 1 1 5B075ADF
-P 4850 6650
-F 0 "R?" V 4850 7000 50  0000 C CNN
-F 1 "33k" V 4850 7150 50  0000 C CNN
-F 2 "" V 4780 6650 50  0001 C CNN
-F 3 "~" H 4850 6650 50  0001 C CNN
-	1    4850 6650
+P 4400 6100
+F 0 "R?" V 4400 6450 50  0000 C CNN
+F 1 "33k" V 4400 6600 50  0000 C CNN
+F 2 "" V 4330 6100 50  0001 C CNN
+F 3 "~" H 4400 6100 50  0001 C CNN
+	1    4400 6100
 	0    -1   -1   0
 $EndComp
@@
 L Device:R R?
 U 1 1 5B075B27
-P 4850 6750
-F 0 "R?" V 4850 7100 50  0000 C CNN
-F 1 "33k" V 4850 7250 50  0000 C CNN
-F 2 "" V 4780 6750 50  0001 C CNN
-F 3 "~" H 4850 6750 50  0001 C CNN
-	1    4850 6750
+P 4400 6200
+F 0 "R?" V 4400 6550 50  0000 C CNN
+F 1 "33k" V 4400 6700 50  0000 C CNN
+F 2 "" V 4330 6200 50  0001 C CNN
+F 3 "~" H 4400 6200 50  0001 C CNN
+	1    4400 6200
 	0    -1   -1   0
 $EndComp
@@
 L Device:R R?
 U 1 1 5B075B6D
-P 4850 6850
-F 0 "R?" V 4850 7200 50  0000 C CNN
-F 1 "33k" V 4850 7350 50  0000 C CNN
-F 2 "" V 4780 6850 50  0001 C CNN
-F 3 "~" H 4850 6850 50  0001 C CNN
-	1    4850 6850
+P 4400 6300
+F 0 "R?" V 4400 6650 50  0000 C CNN
+F 1 "33k" V 4400 6800 50  0000 C CNN
+F 2 "" V 4330 6300 50  0001 C CNN
+F 3 "~" H 4400 6300 50  0001 C CNN
+	1    4400 6300
 	0    -1   -1   0
 $EndComp
@@
 L Device:R R?
 U 1 1 5B075BB5
-P 4850 6950
-F 0 "R?" V 4850 7300 50  0000 C CNN
-F 1 "33k" V 4850 7450 50  0000 C CNN
-F 2 "" V 4780 6950 50  0001 C CNN
-F 3 "~" H 4850 6950 50  0001 C CNN
-	1    4850 6950
+P 4400 6400
+F 0 "R?" V 4400 6750 50  0000 C CNN
+F 1 "33k" V 4400 6900 50  0000 C CNN
+F 2 "" V 4330 6400 50  0001 C CNN
+F 3 "~" H 4400 6400 50  0001 C CNN
+	1    4400 6400
 	0    -1   -1   0
 $EndComp
@@
 L Device:R R?
 U 1 1 5B075BFF
-P 4850 7050
-F 0 "R?" V 4850 7400 50  0000 C CNN
-F 1 "33k" V 4850 7550 50  0000 C CNN
-F 2 "" V 4780 7050 50  0001 C CNN
-F 3 "~" H 4850 7050 50  0001 C CNN
-	1    4850 7050
+P 4400 6500
+F 0 "R?" V 4400 6850 50  0000 C CNN
+F 1 "33k" V 4400 7000 50  0000 C CNN
+F 2 "" V 4330 6500 50  0001 C CNN
+F 3 "~" H 4400 6500 50  0001 C CNN
+	1    4400 6500
 	0    -1   -1   0
 $EndComp
@@
 L Device:R R?
 U 1 1 5B075C4B
-P 4850 7150
-F 0 "R?" V 4850 7500 50  0000 C CNN
-F 1 "33k" V 4850 7650 50  0000 C CNN
-F 2 "" V 4780 7150 50  0001 C CNN
-F 3 "~" H 4850 7150 50  0001 C CNN
-	1    4850 7150
+P 4400 6600
+F 0 "R?" V 4400 6950 50  0000 C CNN
+F 1 "33k" V 4400 7100 50  0000 C CNN
+F 2 "" V 4330 6600 50  0001 C CNN
+F 3 "~" H 4400 6600 50  0001 C CNN
+	1    4400 6600
 	0    -1   -1   0
 $EndComp
@@
 L Device:R R?
 U 1 1 5B075C99
-P 4850 7250
-F 0 "R?" V 4850 7600 50  0000 C CNN
-F 1 "33k" V 4850 7750 50  0000 C CNN
-F 2 "" V 4780 7250 50  0001 C CNN
-F 3 "~" H 4850 7250 50  0001 C CNN
-	1    4850 7250
+P 4400 6700
+F 0 "R?" V 4400 7050 50  0000 C CNN
+F 1 "33k" V 4400 7200 50  0000 C CNN
+F 2 "" V 4330 6700 50  0001 C CNN
+F 3 "~" H 4400 6700 50  0001 C CNN
+	1    4400 6700
 	0    -1   -1   0
 $EndComp
 Wire Wire Line
-	4700 7150 4700 7250
-Connection ~ 4700 7150
-Wire Wire Line
-	4700 7050 4700 7150
-Connection ~ 4700 7050
-Wire Wire Line
-	4700 6950 4700 7050
-Connection ~ 4700 6950
-Wire Wire Line
-	4700 6850 4700 6950
-Connection ~ 4700 6850
-Wire Wire Line
-	4700 6750 4700 6850
-Connection ~ 4700 6750
-Wire Wire Line
-	4700 6650 4700 6750
-Connection ~ 4700 6650
-Wire Wire Line
-	4700 6550 4700 6650
+	4250 6600 4250 6700
+Connection ~ 4250 6600
+Wire Wire Line
+	4250 6500 4250 6600
+Connection ~ 4250 6500
+Wire Wire Line
+	4250 6400 4250 6500
+Connection ~ 4250 6400
+Wire Wire Line
+	4250 6300 4250 6400
+Connection ~ 4250 6300
+Wire Wire Line
+	4250 6200 4250 6300
+Connection ~ 4250 6200
+Wire Wire Line
+	4250 6100 4250 6200
+Connection ~ 4250 6100
+Wire Wire Line
+	4250 6000 4250 6100
 Text GLabel 2050 4550 2    50   Input ~ 0
 3V3_L
@@
 Text GLabel 4700 2550 0    50   Input ~ 0
 3V3_L
-Text GLabel 2600 3250 0    50   Input ~ 0
+Text GLabel 2600 3350 0    50   Input ~ 0
 !Lock
 Wire Wire Line
-	4700 7250 4700 7300
-Connection ~ 4700 7250
+	4250 6700 4250 6750
+Connection ~ 4250 6700
 Wire Wire Line
 	2550 5000 3200 5000
@@
 Wire Wire Line
 	2550 5200 3200 5200
-Text GLabel 5400 6600 0    50   Input ~ 0
+Text GLabel 4950 6050 0    50   Input ~ 0
 mux_p_1
-Text GLabel 5400 6700 0    50   Input ~ 0
+Text GLabel 4950 6150 0    50   Input ~ 0
 mux_p_2
-Text GLabel 5400 6900 0    50   Input ~ 0
+Text GLabel 4950 6350 0    50   Input ~ 0
 mux_p_4
-Text GLabel 5400 6800 0    50   Input ~ 0
+Text GLabel 4950 6250 0    50   Input ~ 0
 mux_p_3
-Text GLabel 5400 7000 0    50   Input ~ 0
+Text GLabel 4950 6450 0    50   Input ~ 0
 mux_p_5
-Text GLabel 5400 7100 0    50   Input ~ 0
+Text GLabel 4950 6550 0    50   Input ~ 0
 mux_p_6
-Text GLabel 5400 7200 0    50   Input ~ 0
+Text GLabel 4950 6650 0    50   Input ~ 0
 mux_p_7
 Wire Wire Line
-	5400 6550 5400 6500
-Wire Wire Line
-	5000 6550 5400 6550
-Wire Wire Line
-	5400 6600 5400 6650
-Wire Wire Line
-	5000 6650 5400 6650
-Wire Wire Line
-	5400 6750 5400 6700
-Wire Wire Line
-	5000 6750 5400 6750
-Wire Wire Line
-	5000 6850 5400 6850
-Wire Wire Line
-	5400 6850 5400 6800
-Wire Wire Line
-	5400 6950 5400 6900
-Wire Wire Line
-	5000 6950 5400 6950
-Wire Wire Line
-	5400 7050 5400 7000
-Wire Wire Line
-	5000 7050 5400 7050
-Wire Wire Line
-	5400 7150 5400 7100
-Wire Wire Line
-	5000 7150 5400 7150
-Wire Wire Line
-	5400 7250 5400 7200
-Wire Wire Line
-	5000 7250 5400 7250
+	4950 6000 4950 5950
+Wire Wire Line
+	4550 6000 4950 6000
+Wire Wire Line
+	4950 6050 4950 6100
+Wire Wire Line
+	4550 6100 4950 6100
+Wire Wire Line
+	4950 6200 4950 6150
+Wire Wire Line
+	4550 6200 4950 6200
+Wire Wire Line
+	4550 6300 4950 6300
+Wire Wire Line
+	4950 6300 4950 6250
+Wire Wire Line
+	4950 6400 4950 6350
+Wire Wire Line
+	4550 6400 4950 6400
+Wire Wire Line
+	4950 6500 4950 6450
+Wire Wire Line
+	4550 6500 4950 6500
+Wire Wire Line
+	4950 6600 4950 6550
+Wire Wire Line
+	4550 6600 4950 6600
+Wire Wire Line
+	4950 6700 4950 6650
+Wire Wire Line
+	4550 6700 4950 6700
 Text GLabel 5850 4850 0    50   Input ~ 0
 mux_p_0
-Text GLabel 5400 6500 0    50   Input ~ 0
+Text GLabel 4950 5950 0    50   Input ~ 0
 mux_p_0
 Text GLabel 7250 4850 0    50   Input ~ 0
@@
 Text GLabel 5850 5800 0    50   Input ~ 0
 mux_p_4
+Text GLabel 2950 3200 0    50   Input ~ 0
+GPIO0
+Wire Wire Line
+	2650 3300 2650 3100
+Connection ~ 2650 3100
+Wire Wire Line
+	2600 3350 2950 3350
+Wire Wire Line
+	2950 3350 2950 3300
+Connection ~ 2950 3300
 $EndSCHEMATC
